Commit message: using aruco markers for signal

File: src/world_simulation/models/block/block_placeholder.urdf (robot description, URDF)
Before this commit: robot block_placeholder, 4 links, 3 joints
Links:
- link block_placeholder_0: mass .1 -> 500
- link block_placeholder_1: mass .1 -> 500
- link block_placeholder_2: mass .1 -> 500
- link block_placeholder_3: mass .1 -> 500
