Commit message: block is now a big boi, can be seen from further away

File: src/world_simulation/models/block/block_signal.urdf (robot description, URDF)
Before this commit: robot block, 3 links, 2 joints
Links:
- link handhold_1: geometry collision box size=0.2 0.2 0.01; visual mesh filename=package://world_simulation/models/aruco_cube/meshes/aruco_c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 scale=2 2 .1
- link handhold_2: mass .2 -> 5; geometry collision box size=0.08 0.08 0.01; visual mesh filename=package://world_simulation/models/aruco_cube/meshes/aruco_c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 scale=.8 .8 .1
Joints:
- joint block_to_handholds_1: origin xyz=0 0 0.155 -> xyz=0 0 0.2
- joint block_to_handholds_2: origin xyz=0 0 -0.15 -> xyz=0 0 -0.2
