Commit message: added package to support setting autonavigation goals

File: src/world_simulation/models/block/block.urdf (robot description, URDF)
Before this commit: robot block, 1 links, 0 joints
Links:
- link block: geometry collision box size=0.2 0.2 0.2; visual box size=0.2 0.2 0.2

Commit message: changing block size back to 0.045

File: src/world_simulation/models/block/block.urdf (robot description, URDF)
Before this commit: robot block, 1 links, 0 joints
Links:
- link block: geometry collision box size=0.045 0.045 0.045; visual box size=0.045 0.045 0.045

Commit message: removed block_size constant in favor of using block size parsed from block.urdf spec, refactored square structure logic into WorldSimulation

File: src/world_simulation/models/block/block.urdf (robot description, URDF)
Before this commit: robot block, 1 links, 0 joints
Links:
- link block: geometry collision box size=0.06 0.06 0.12; visual box size=0.06 0.06 0.12

Commit message: reading in block mass from block_urdf spec, calculating block inertia in code

File: src/world_simulation/models/block/block.urdf (robot description, URDF)
Before this commit: robot block, 1 links, 0 joints
Links:
- link block: mass 0.5 -> 1

Commit message: making block lighter

File: src/world_simulation/models/block/block.urdf (robot description, URDF)
Before this commit: robot block, 1 links, 0 joints
Links:
- link block: mass 1 -> .01

Commit message: picking up blocks with Aruco

File: src/world_simulation/models/block/block.urdf (robot description, URDF)
Before this commit: robot block, 1 links, 0 joints
Links:
- link block: mass .01 -> .05; geometry collision box size=0.055 0.055 0.33; visual mesh filename=package://world_simulation/models/aruco_cube/meshes/aruco_c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 scale=1 1 6

Commit message: extended planner cuz aruco friggen SUCKS

File: src/world_simulation/models/block/block.urdf (robot description, URDF)
Before this commit: robot block, 1 links, 0 joints
Links:
- link block: geometry collision box size=0.05 0.05 0.40; visual mesh filename=package://world_simulation/models/aruco_cube/meshes/aruco_c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 scale=1 1 8

Commit message: different colors for exploration world and structure world

File: src/world_simulation/models/block/block.urdf (robot description, URDF)
Before this commit: robot block, 1 links, 0 joints
Links:
- link block: geometry collision box size=0.05 0.05 0.40

Commit message: added love handles

File: src/world_simulation/models/block/block.urdf (robot description, URDF)
Before this commit: robot block, 1 links, 0 joints
Links:
- added link handholds, mass .01; collision box size=0.1 0.1 0.02; visual box size=0.1 0.1 0.02
- link block: mass .05 -> .01
Joints:
- added joint block_to_handholds: type fixed, parent block, child handholds, origin xyz=0 0 0.1

Commit message: dumbell block and lower placement

File: src/world_simulation/models/block/block.urdf (robot description, URDF)
Before this commit: robot block, 2 links, 1 joints
Links:
- removed link handholds
- added link handhold_1, mass .01; collision box size=0.05 0.05 0.1
- added link handhold_2, mass .01; collision box size=0.05 0.05 0.1
- link block: geometry collision box size=0.03 0.03 0.40; visual box size=0.03 0.03 0.4
Joints:
- removed joint block_to_handholds
- added joint block_to_handholds_1: type fixed, parent block, child handhold_1, origin xyz=0 0 0.15
- added joint block_to_handholds_2: type fixed, parent block, child handhold_2, origin xyz=0 0 -0.15

Commit message: separated exploration and structure block urdf files, added call to take photos in world simulation

File: src/world_simulation/models/block/block.urdf (robot description, URDF)
Before this commit: robot block, 3 links, 2 joints
Links:
- link handhold_1: geometry collision box size=0.05 0.05 0.1; visual mesh filename=package://world_simulation/models/aruco_cube/meshes/aruco_c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 scale=1 1 2

Commit message: put block.urdf file back so it works again

File: src/world_simulation/models/block/block.urdf (robot description, URDF)
Before this commit: robot block, 3 links, 2 joints
Links:
- link handhold_2: geometry collision box size=0.05 0.05 0.1; visual mesh filename=package://world_simulation/models/aruco_cube/meshes/aruco_c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 scale=1 1 2

Commit message: everything put together

File: src/world_simulation/models/block/block.urdf (robot description, URDF)
Before this commit: robot block, 3 links, 2 joints
Links:
- link handhold_2: mass .01 -> .1
Joints:
- joint block_to_handholds_1: origin xyz=0 0 0.15 -> xyz=0 0 0.155

Commit message: adding placeholder urdf

File: src/world_simulation/models/block/block.urdf (robot description, URDF)
Before this commit: robot block, 3 links, 2 joints
Links:
- link handhold_2: geometry collision box size=0.04 0.04 0.1; visual mesh filename=package://world_simulation/models/aruco_cube/meshes/aruco_c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 scale=.8 .8 2

File: src/world_simulation/models/block/block_placeholder.urdf (robot description, URDF)
Before this commit: robot block_placeholder, 4 links, 4 joints
Links:
- link block_placeholder_0: geometry collision box size=0.005 0.05 0.04; visual box size=0.005 0.05 0.04
- link block_placeholder_1: geometry collision box size=0.005 0.05 0.04; visual box size=0.005 0.05 0.04
- link block_placeholder_2: geometry collision box size=0.05 0.005 0.04; visual box size=0.05 0.005 0.04
- link block_placeholder_3: geometry collision box size=0.05 0.005 0.04; visual box size=0.05 0.005 0.04
Joints:
- removed joint 2_to_1

Commit message: we close

File: src/world_simulation/models/block/block.urdf (robot description, URDF)
Before this commit: robot block, 3 links, 2 joints
Links:
- link block: geometry collision box size=0.03 0.03 0.3; visual box size=0.03 0.03 0.3
- link handhold_1: geometry collision box size=0.09 0.09 0.05; visual mesh filename=package://world_simulation/models/aruco_cube/meshes/aruco_c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 scale=1.8 1.8 1
- link handhold_2: geometry collision box size=0.09 0.09 0.05; visual mesh filename=package://world_simulation/models/aruco_cube/meshes/aruco_c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 scale=1.8 1.8 1

File: src/world_simulation/models/block/block_placeholder.urdf (robot description, URDF)
Before this commit: robot block_placeholder, 4 links, 3 joints
Links:
- removed link block_placeholder_0
- removed link block_placeholder_1
- removed link block_placeholder_2
- removed link block_placeholder_3
- added link block_placeholder_aruco, mass 500; collision box size=0.09 0.09 0.005; visual mesh filename=package://world_simulation/models/aruco_cube/meshes/aruco_c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 scale=1.125 1.125 .1
Joints:
- removed joint 0_to_2
- removed joint 0_to_3
- removed joint 3_to_1
