Commit message: more stable structure and images/schematic of it

File: src/world_simulation/models/block/structure_block.urdf (robot description, URDF)
Before this commit: robot block, 1 links, 0 joints
Links:
- link block: mass .01 -> .5

Commit message: imaging with new block sizes

File: src/world_simulation/models/block/structure_block.urdf (robot description, URDF)
Before this commit: robot block, 1 links, 0 joints
Links:
- link block: geometry collision box size=0.09 0.09 0.355; visual box size=0.09 0.09 0.355

Commit message: increasing structure block mass from 0.5 to 100 to avoid falling

File: src/world_simulation/models/block/structure_block.urdf (robot description, URDF)
Before this commit: robot block, 1 links, 0 joints
Links:
- link block: mass .5 -> 100
