Commit message: clean up codeeee

File: src/world_simulation/models/block/aruco_block.urdf (robot description, URDF)
Before this commit: robot block, 3 links, 2 joints
Links:
- link block: geometry collision box size=0.03 0.03 0.4; visual box size=0.03 0.03 0.4
Joints:
- joint block_to_handholds_1: origin xyz=0 0 0.155 -> xyz=0 0 0.205
- joint block_to_handholds_2: origin xyz=0 0 -0.15 -> xyz=0 0 -0.20

File: src/world_simulation/models/block/block_placeholder.urdf (robot description, URDF)
Before this commit: robot block_placeholder, 1 links, 0 joints
Links:
- link block_placeholder_aruco: geometry collision box size=0.09 0.09 0.0001; visual mesh filename=package://world_simulation/models/aruco_cube/meshes/aruco_c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 scale=1.125 1.125 .002
